File: PCB/M4ROM_27256.kicad_sch (KiCad schematic)
At the start: 7 parts, among them J1 32Kx8_mask_rom_socket, J2 4ROM_prog_female, SW1 CUS-14TB, U1 29F010

Commit message: pcb polish
Parts:
- SW1: footprint 000_LOCAL:SW_SP4T_CUS-14B -> 000_LOCAL:SW_SP4T_CUS-14B - PTH; symbol 0_LOCAL:SW_1P4T_CUS-14B -> 000_LOCAL:SW_1P4T_CUS-14B_-_PTH
Connections:
- net GND: now also SW1.M
Changed lines of the file:
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@@
   (title_block
     (title "M4ROM 27256")
-    (date "2023-12-30")
-    (rev "003")
+    (date "2023-12-31")
+    (rev "004")
     (company "Brian K. White b.kenyon.w@gmail.com")
     (comment 1 "CC-BY-SA")
@@
   (junction (at 152.4 119.38) (diameter 0) (color 0 0 0 0)
   )
+  (junction (at 62.23 166.37) (diameter 0) (color 0 0 0 0)
+  )
   (junction (at 101.6 154.94) (diameter 0) (color 0 0 0 0)
   )
@@
     (stroke (width 0) (type default))
   )
+  (wire (pts (xy 59.69 166.37) (xy 62.23 166.37))
+    (stroke (width 0) (type default))
+  )
   (wire (pts (xy 92.71 161.29) (xy 93.98 161.29))
     (stroke (width 0) (type default))
@@
   )
   (text "Castellated edge contacts\nto fit Molex 78805 socket\nwith 32Kx8 mask rom pinout\n(27256 without VPP)"
-    (at 67.31 53.34 0)
+    (at 67.31 49.53 0)
     (effects (font (size 2 2)) (justify left bottom))
   )
@@
       (effects (font (size 1.27 1.27)))
     )
-    (property "Value" "32Kx8_mask_rom_socket" (at 89.662 62.23 0)
+    (property "Value" "32Kx8_mask_rom_socket" (at 77.47 53.34 0)
       (effects (font (size 1.27 1.27)) (justify left))
     )
@@
     )
   )
-  (symbol (lib_id "0_LOCAL:SW_1P4T_CUS-14B") (at 60.96 160.02 0) (unit 1)
+  (symbol (lib_id "000_LOCAL:SW_1P4T_CUS-14B_-_PTH") (at 60.96 160.02 0) (unit 1)
     (in_bom yes) (on_board yes) (dnp no)
     (property "Reference" "SW1" (at 62.23 153.67 0)
@@
       (effects (font (size 1.27 1.27)))
     )
-    (property "Footprint" "000_LOCAL:SW_SP4T_CUS-14B" (at 45.085 155.575 0)
+    (property "Footprint" "000_LOCAL:SW_SP4T_CUS-14B - PTH" (at 45.085 155.575 0)
       (effects (font (size 1.27 1.27)) hide)
     )
@@
     (pin "6")
     (pin "S")
+    (pin "M")
     (instances
       (project "WP-2_IC-Card_MRAM_512"
@@
     )
   )
-  (symbol (lib_id "0_LOCAL:GND") (at 60.96 166.37 0) (mirror y) (unit 1)
-    (in_bom yes) (on_board yes) (dnp no)
-    (property "Reference" "#PWR020" (at 60.96 170.18 0)
-      (effects (font (size 1.27 1.27)) hide)
-    )
-    (property "Value" "GND" (at 60.96 170.18 0)
-      (effects (font (size 1.27 1.27)) hide)
-    )
-    (property "Footprint" "" (at 60.96 166.37 0)
-      (effects (font (size 1.27 1.27)) hide)
-    )
-    (property "Datasheet" "" (at 60.96 166.37 0)
-      (effects (font (size 1.27 1.27)) hide)
-    )
+  (symbol (lib_id "0_LOCAL:GND") (at 62.23 166.37 0) (mirror y) (unit 1)
+    (in_bom yes) (on_board yes) (dnp no)
+    (property "Reference" "#PWR020" (at 62.23 170.18 0)
+      (effects (font (size 1.27 1.27)) hide)
+    )
+    (property "Value" "GND" (at 62.23 170.18 0)
+      (effects (font (size 1.27 1.27)) hide)
+    )
+    (property "Footprint" "" (at 62.23 166.37 0)
+      (effects (font (size 1.27 1.27)) hide)
+    )
+    (property "Datasheet" "" (at 62.23 166.37 0)
+      (effects (font (size 1.27 1.27)) hide)
+    )
