File: PCB/M4ROM_TANDY.kicad_sch (KiCad schematic)
At the start: 7 parts, among them J1 Tandy_100_102_200_option_rom, J2 4ROM_prog_female, SW1 CUS-14TB, U1 29F010

Commit message: pcb polish
Parts:
- SW1: footprint 000_LOCAL:SW_SP4T_CUS-14B -> 000_LOCAL:SW_SP4T_CUS-14B - PTH; symbol 0_LOCAL:SW_1P4T_CUS-14B -> 000_LOCAL:SW_1P4T_CUS-14B_-_PTH
Connections:
- net GND: now also SW1.M
Changed lines of the file:
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@@
   (title_block
     (title "M4ROM TANDY")
-    (date "2023-12-30")
-    (rev "006")
+    (date "2023-12-31")
+    (rev "008")
     (company "Brian K. White b.kenyon.w@gmail.com")
     (comment 1 "CC-BY-SA")
@@
   (junction (at 85.09 156.21) (diameter 0) (color 0 0 0 0)
   )
+  (junction (at 62.23 170.18) (diameter 0) (color 0 0 0 0)
+  )
   (no_connect (at 66.04 160.02))
   (no_connect (at 78.74 106.68))
@@
   )
   (wire (pts (xy 66.04 162.56) (xy 77.47 162.56))
+    (stroke (width 0) (type default))
+  )
+  (wire (pts (xy 59.69 170.18) (xy 62.23 170.18))
     (stroke (width 0) (type default))
   )
@@
     (pin "6")
     (instances
-      (project "4ROM_100"
+      (project "M4ROM_TANDY"
         (path "/c6d91437-1142-48a2-b1d0-d6e4e1e576c8"
           (reference "U1") (unit 1)
@@
     (pin "9")
     (instances
-      (project "4ROM_100"
+      (project "M4ROM_TANDY"
         (path "/c6d91437-1142-48a2-b1d0-d6e4e1e576c8"
           (reference "J1") (unit 1)
@@
     (pin "1")
     (instances
-      (project "4ROM_100"
+      (project "M4ROM_TANDY"
         (path "/c6d91437-1142-48a2-b1d0-d6e4e1e576c8"
           (reference "#PWR0101") (unit 1)
@@
     (pin "1")
     (instances
-      (project "4ROM_100"
+      (project "M4ROM_TANDY"
         (path "/c6d91437-1142-48a2-b1d0-d6e4e1e576c8"
           (reference "#PWR0102") (unit 1)
@@
     (pin "1")
     (instances
-      (project "4ROM_100"
+      (project "M4ROM_TANDY"
         (path "/c6d91437-1142-48a2-b1d0-d6e4e1e576c8"
           (reference "#PWR0105") (unit 1)
@@
         )
       )
-      (project "4ROM_100"
+      (project "M4ROM_TANDY"
         (path "/c6d91437-1142-48a2-b1d0-d6e4e1e576c8"
           (reference "#PWR06") (unit 1)
@@
     (pin "1")
     (instances
-      (project "4ROM_100"
+      (project "M4ROM_TANDY"
         (path "/c6d91437-1142-48a2-b1d0-d6e4e1e576c8"
           (reference "#PWR01") (unit 1)
@@
         )
       )
-      (project "4ROM_100"
+      (project "M4ROM_TANDY"
         (path "/c6d91437-1142-48a2-b1d0-d6e4e1e576c8"
           (reference "#PWR09") (unit 1)
@@
     (pin "1")
     (instances
-      (project "4ROM_100"
+      (project "M4ROM_TANDY"
         (path "/c6d91437-1142-48a2-b1d0-d6e4e1e576c8"
           (reference "#PWR0116") (unit 1)
@@
         )
       )
-      (project "4ROM_100"
+      (project "M4ROM_TANDY"
         (path "/c6d91437-1142-48a2-b1d0-d6e4e1e576c8"
           (reference "#PWR04") (unit 1)
@@
     (pin "5")
     (instances
-      (project "4ROM_100"
+      (project "M4ROM_TANDY"
         (path "/c6d91437-1142-48a2-b1d0-d6e4e1e576c8"
           (reference "RA1") (unit 4)
@@
         )
       )
-      (project "4ROM_100"
+      (project "M4ROM_TANDY"
         (path "/c6d91437-1142-48a2-b1d0-d6e4e1e576c8"
           (reference "#PWR07") (unit 1)
@@
         )
       )
-      (project "4ROM_100"
+      (project "M4ROM_TANDY"
         (path "/c6d91437-1142-48a2-b1d0-d6e4e1e576c8"
           (reference "D1") (unit 2)
@@
     )
   )
-  (symbol (lib_id "0_LOCAL:SW_1P4T_CUS-14B") (at 60.96 163.83 0) (unit 1)
+  (symbol (lib_id "000_LOCAL:SW_1P4T_CUS-14B_-_PTH") (at 60.96 163.83 0) (unit 1)
     (in_bom yes) (on_board yes) (dnp no)
     (property "Reference" "SW1" (at 62.23 157.48 0)
@@
       (effects (font (size 1.27 1.27)))
     )
-    (property "Footprint" "000_LOCAL:SW_SP4T_CUS-14B" (at 45.085 159.385 0)
+    (property "Footprint" "000_LOCAL:SW_SP4T_CUS-14B - PTH" (at 45.085 159.385 0)
       (effects (font (size 1.27 1.27)) hide)
     )
@@
     (pin "6")
     (pin "S")
+    (pin "M")
     (instances
       (project "WP-2_IC-Card_MRAM_512"
@@
         )
       )
-      (project "4ROM_100"
+      (project "M4ROM_TANDY"
         (path "/c6d91437-1142-48a2-b1d0-d6e4e1e576c8"
           (reference "SW1") (unit 1)
@@
     (pin "2")
     (instances
-      (project "4ROM_100"
+      (project "M4ROM_TANDY"
         (path "/c6d91437-1142-48a2-b1d0-d6e4e1e576c8"
           (reference "C1") (unit 1)
@@
     (pin "5")
     (instances
-      (project "4ROM_100"
+      (project "M4ROM_TANDY"
         (path "/c6d91437-1142-48a2-b1d0-d6e4e1e576c8"
           (reference "RA1") (unit 1)
@@
         )
       )
-      (project "4ROM_100"
+      (project "M4ROM_TANDY"
         (path "/c6d91437-1142-48a2-b1d0-d6e4e1e576c8"
           (reference "#PWR03") (unit 1)
@@
         )
       )
-      (project "4ROM_100"
+      (project "M4ROM_TANDY"
         (path "/c6d91437-1142-48a2-b1d0-d6e4e1e576c8"
           (reference "D1") (unit 1)
@@
     (pin "5")
     (instances
-      (project "4ROM_100"
+      (project "M4ROM_TANDY"
         (path "/c6d91437-1142-48a2-b1d0-d6e4e1e576c8"
           (reference "RA1") (unit 3)
@@
     (pin "1")
     (instances
-      (project "4ROM_100"
+      (project "M4ROM_TANDY"
         (path "/c6d91437-1142-48a2-b1d0-d6e4e1e576c8"
           (reference "#PWR0110") (unit 1)
@@
     (pin "9")
     (instances
-      (project "4ROM_100"
+      (project "M4ROM_TANDY"
         (path "/c6d91437-1142-48a2-b1d0-d6e4e1e576c8"
           (reference "J2") (unit 1)
@@
     (pin "5")
     (instances
-      (project "4ROM_100"
+      (project "M4ROM_TANDY"
         (path "/c6d91437-1142-48a2-b1d0-d6e4e1e576c8"
           (reference "RA1") (unit 2)
@@
         )
       )
-      (project "4ROM_100"
+      (project "M4ROM_TANDY"
         (path "/c6d91437-1142-48a2-b1d0-d6e4e1e576c8"
           (reference "#PWR05") (unit 1)
@@
     )
   )
-  (symbol (lib_id "0_LOCAL:GND") (at 60.96 170.18 0) (mirror y) (unit 1)
-    (in_bom yes) (on_board yes) (dnp no)
-    (property "Reference" "#PWR020" (at 60.96 173.99 0)
-      (effects (font (size 1.27 1.27)) hide)
-    )
-    (property "Value" "GND" (at 60.96 173.99 0)
-      (effects (font (size 1.27 1.27)) hide)
-    )
-    (property "Footprint" "" (at 60.96 170.18 0)
-      (effects (font (size 1.27 1.27)) hide)
-    )
-    (property "Datasheet" "" (at 60.96 170.18 0)
+  (symbol (lib_id "0_LOCAL:GND") (at 62.23 170.18 0) (mirror y) (unit 1)
+    (in_bom yes) (on_board yes) (dnp no)
+    (property "Reference" "#PWR020" (at 62.23 173.99 0)
+      (effects (font (size 1.27 1.27)) hide)
+    )
+    (property "Value" "GND" (at 62.23 173.99 0)
+      (effects (font (size 1.27 1.27)) hide)
+    )
+    (property "Footprint" "" (at 62.23 170.18 0)
+      (effects (font (size 1.27 1.27)) hide)
+    )
+    (property "Datasheet" "" (at 62.23 170.18 0)
       (effects (font (size 1.27 1.27)) hide)
     )
@@
         )
       )
-      (project "4ROM_100"
+      (project "M4ROM_TANDY"
         (path "/c6d91437-1142-48a2-b1d0-d6e4e1e576c8"
           (reference "#PWR02") (unit 1)
