File: PCB/M4ROM_27256.kicad_pcb (KiCad board)
At the start: 2 copper layers, 38 x 16.6 mm, 7 parts, among them J1 32Kx8_mask_rom_socket, J2 4ROM_prog_female, SW1 CUS-14TB, U1 29F010

Commit message: readme. fillet tracks
Routing:
- net GND: vias 34 -> 36

Commit message: simpler diodes
Parts:
- D1: value BAV70S -> BAW56; footprint 000_LOCAL:TSSOP-6-symmetric -> 000_LOCAL:SOT-23
- moved D1 0.69 mm to (132.7, 94.6), turned to 90 degrees
Connections:
- D1 pad 1: /BANK_2 -> /A16
- D1 pad 2: /BANK_3 -> /A15
- D1 pad 3: /A16 -> /BANK_4
- SW1 pad 2: /BANK_2 -> /A15
- SW1 pad 5: /BANK_3 -> /A16
Routing:
- net /BANK_3: track 37.3 -> 0.00 mm, vias 2 -> 0
- net /BANK_2: track 33.3 -> 0.00 mm, vias 2 -> 0
- net /A15: track 10.4 -> 38.6 mm, vias 2 -> 3
- net /A16: track 13.9 -> 38.1 mm, vias 2 -> 4
- net /BANK_4: track 39.1 -> 41.2 mm
- net VCC: track 45.2 -> 44.0 mm
- net /A12: track 16.1 -> 16.8 mm
- net GND: vias 36 -> 39
