File: PCB/M4ROM_TANDY.kicad_pcb (KiCad board)
At the start: 2 copper layers, 38 x 16.6 mm, 7 parts, among them J1 Tandy_100_102_200_option_rom, J2 4ROM_prog_female, SW1 CUS-14TB, U1 29F010

Commit message: readme. fillet tracks
Routing:
- net /A10: track 34.9 -> 32.9 mm
- net /~{OE}: track 16.2 -> 14.9 mm
- net /A4: track 13.5 -> 12.7 mm
- net GND: vias 34 -> 42

Commit message: simpler diodes
Parts:
- D1: value BAV70S -> BAW56; footprint 000_LOCAL:TSSOP-6-symmetric -> 000_LOCAL:SOT-23
- moved D1 0.79 mm to (132.5, 94.1), turned to 90 degrees
Connections:
- D1 pad 1: /BANK_2 -> /A16
- D1 pad 2: /BANK_3 -> /A15
- D1 pad 3: /A16 -> /BANK_4
- SW1 pad 2: /BANK_2 -> /A15
- SW1 pad 5: /BANK_3 -> /A16
- U1 pad 10: /A16 -> /A15
- U1 pad 11: /A15 -> /A16
Routing:
- net /BANK_3: track 35.7 -> 0.00 mm, vias 4 -> 0
- net /BANK_2: track 32.8 -> 0.00 mm, vias 4 -> 0
- net /A15: track 10.6 -> 37.2 mm, vias 2 -> 4
- net /A16: track 14.5 -> 37.2 mm, vias 2 -> 4
- net /BANK_4: track 39.2 -> 41.6 mm
- net VCC: track 42.2 -> 43.7 mm
- net GND: vias 42 -> 51
